File: SOURCES/kiCAD/FreeDSP_OCTAVIA.kicad_pcb (KiCad board)
At the start: 2 copper layers, 178 x 99 mm, 492 parts, among them IC1 TPS5430DDA, IC2 PCM1808QPWRQ1, J1 Conn_01x08, J11 Conn_Coaxial, J12 IDC_2x5, J13 Conn_01x05, J16 MJ-519, J17 MJ-519, J2 DC12V-IN, J20 MJ-519, J21 MJ-519, J24 Header6P, J25 Conn_01x06, J27 Conn_01x06, J28 Header6P, J3 Conn_01x08, J4 Header_01x06, J5 Conn_Coaxial_x2, J6 8P_DIP_SOCKET, J8 Header_01x04, P1 Conn_02x20_Odd_Even, Q1 AO3401A, Q10 2SC3326, Q11 2SC3326, Q12 MJD45H11T4, Q13 2N7002, Q14 2N7002, Q15 2SC3326, Q16 2SC3326, Q17 2SC3326, Q18 2SC3326, Q19 2SC3326, Q2 MMBT5401, Q20 2SC3326, Q21 2SC3326, Q22 2SC3326, Q23 2SC3326, Q24 2SC3326, Q25 2SC3326, Q26 2SC3326, Q27 2SC3326, Q28 2SC3326, Q29 AO3401A, Q3 2N7002, Q30 2N7002, Q31 2N7002, Q4 MMBT5401, Q5 AO3401A, Q6 2N7002, Q7 AO3401A, Q8 2N7002, Q9 2N7002, SW1 SW_Push, SW2 SW_SPDT, SW3 SW_SPDT, SW4 SW_NOP_DPDT, SW7 DSP_RES, T1 PE-65612NL, U1 GP1UXC41QS, U10 74LVC1G86, U11 74LVC1G04, U12 ADAU1452, U13 25LC_1024, U14 PCM5102A, U15 74LVC1G04, U16 PCM5102A, U17 PCM5102A, U18 PCM5102A, U2 PLR135-T10, U20 OPA1632DR, U21 OPA1632DR, U22 OPA1632DR, U23 OPA1632DR, U24 OPA1632DR, U25 OPA1632DR, U26 OPA1632DR, U27 OPA1632DR, U3 AMS1117-5.0, U4 PLT133-T10W, U5 TPS5430DDA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

Commit message: Updated version0.2
Parts:
- removed the Z2 at (109.5, 45.9)
- JP2: footprint Jumper:SolderJumper-2_P1.3mm_Open_RoundedPad1.0x1.5mm -> Jumper:SolderJumper-2_P1.3mm_Bridged_RoundedPad1.0x1.5mm
- renumbered G*** to Z2
Other:
- board text added: "10"
- board text added: "20"
- board text added: "30"
- board text added: "40"
- board text added: "OPT-OUT"
- board text added: "ROM SELECT"
- board text added: "Rev. 0.2"
- board text removed: "BOOT SELECT"
- board text removed: "OUT-OUT"
- board text removed: "Rev. 0.1"

Commit message: Version0.2 Board. Reviced PCB design.
Parts:
- added C140: 0.1uF, Capacitor_SMD:C_0805_2012Metric_Pad1.18x1.45mm_HandSolder, F.Cu at (144.1, 93.8)
- added D22: 1N4148W, Diode_SMD:D_SOD-123, F.Cu at (150.7, 96.4)
- added D23: 1N4148W, Diode_SMD:D_SOD-123, F.Cu at (158.1, 79.5)
- added J10: Conn_01x02, Connector_PinHeader_2.54mm:PinHeader_1x02_P2.54mm_Vertical, F.Cu at (54.0, 55.5)
- added J7: Header_01x04, Connector_PinHeader_2.54mm:PinHeader_1x04_P2.54mm_Vertical, F.Cu at (180.4, 60.4)
- added J9: Conn_01x02, Connector_PinHeader_2.54mm:PinHeader_1x02_P2.54mm_Vertical, F.Cu at (94.5, 55.5)
- added Q32: 2N7002, Package_TO_SOT_SMD:SOT-23_Handsoldering, F.Cu at (151.6, 75.3)
- added R49: 3.3k, Resistor_SMD:R_0603_1608Metric, F.Cu at (158.3, 58.9)
- added R50: 10k, Resistor_SMD:R_0805_2012Metric_Pad1.20x1.40mm_HandSolder, F.Cu at (154.7, 78.3)
- added R51: 100k, Resistor_SMD:R_0805_2012Metric_Pad1.20x1.40mm_HandSolder, F.Cu at (161.5, 95.7)
- added TP1: TestPoint_GNDA, TestPoint:TestPoint_THTPad_2.0x2.0mm_Drill1.0mm, F.Cu at (112.6, 128.3)
- added TP2: TestPoint_DGND, TestPoint:TestPoint_THTPad_2.0x2.0mm_Drill1.0mm, F.Cu at (157.9, 101.9)
- C13: footprint Capacitor_THT:CP_Radial_D5.0mm_P2.00mm -> Capacitor_THT:CP_Radial_D10.0mm_P2.50mm_P5.00mm
- JP2: value Jumper_NO -> Jumper_NC
- R100, R101, R102, R103: value 330R -> 1k
- R33, R7: value 1k -> 3.3k
- R76: value 3.3k -> 330R
- R92, R94: value 100 -> 100R
- SW1, SW7: footprint OPL_Switch:SW2-5.0-6.0X3.0X4.3MM -> Button_Switch_THT:SW_Tactile_SPST_Angled_PTS645Vx83-2LFS
- U13: value 25LC_1024 -> 25AA1024
- moved SW7 108.0 mm to (32.7, 108.1), turned to 90 degrees
- moved D13 23.0 mm to (154.9, 60.9)
- moved C13 15.3 mm to (113.9, 110.4), turned to 0 degrees
- moved R108 12.0 mm to (159.1, 65.8), turned to 270 degrees
- moved Q3 11.2 mm to (193.0, 57.3)
- moved D3 11.0 mm to (192.9, 52.9)
- moved R29 7.56 mm to (123.7, 115.9)
- moved R98 4.56 mm to (54.5, 61.1)
- moved FB6 4.14 mm to (39.8, 106.5), turned to 180 degrees
- moved R96 3.54 mm to (91.4, 59.0)
- moved R176 3.54 mm to (118.8, 116.3)
- moved Z2 2.82 mm to (183.5, 92.9)
- moved D12 2.52 mm to (162.5, 77.4)
- moved R16 2.31 mm to (184.0, 60.5), turned to 270 degrees
- moved R12 1.95 mm to (153.3, 58.2)
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Connections:
- D12 pad 1: USB_MUTE -> Net-(D12-Pad1)
- D13 pad 1: USB_MUTE -> Net-(D12-Pad1)
- D13 pad 2: Net-(A1-Pad11) -> Net-(D13-Pad2)
- J13 pad 1: +5V -> +3V3
- J13 pad 2: Net-(J13-Pad2) -> ~SEL_USB
- J8 pad 2: RP_SDA -> +3.3VP
- J8 pad 4: +3.3VP -> RP_SDA
- Q14 pad 1: USB_MUTE -> Net-(A1-Pad11)
- Q14 pad 3: AUX5 -> Net-(D13-Pad2)
- Q9 pad 1: MUTE -> Net-(D22-Pad1)
- R100 pad 2: Net-(J13-Pad2) -> ~SEL_USB
- R108 pad 1: GND -> +3V3
- R108 pad 2: USB_MUTE -> ~SEL_USB
Routing:
- net Net-(D22-Pad1): track 0.00 -> 52.4 mm, vias 0 -> 4
- net Net-(A1-Pad11): track 9.52 -> 39.3 mm
- net GNDA: track 380.5 -> 409.2 mm, vias 27 -> 29
- net USB_MUTE: track 27.7 -> 0.00 mm
- net Net-(D12-Pad1): track 0.00 -> 25.1 mm
- net ~DSP-RESET: track 124.7 -> 145.3 mm, vias 3 -> 4
- net ~SEL_USB: track 0.00 -> 19.4 mm
- net MUTE: track 253.3 -> 271.6 mm, vias 14 -> 12
- net Net-(D3-Pad4): track 2.21 -> 17.9 mm
- net AUX5: track 131.8 -> 116.3 mm
- net +5VA: track 190.2 -> 176.8 mm, vias 9 -> 51
- net +3V3: track 708.4 -> 719.3 mm
- net Net-(D3-Pad3): track 12.9 -> 23.4 mm, vias 0 -> 1
- net Net-(D3-Pad1): track 15.2 -> 24.3 mm
- net BCK_IN0: track 51.2 -> 59.2 mm
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- added copper zone on B.Cu, net +3.3VA
- added copper zone on F.Cu, net +3.3VA
- added copper zone on B.Cu, net +5VA
- added copper zone on F.Cu, net +5VA
Other:
- board text added: "+1.2V"
- board text added: "+5"
- board text added: "-5"
- board text added: "12V"
- board text added: "20%"
- board text added: "24.576MHz"
- board text added: "3.3"
- board text added: "40%"
- board text added: "6.5V-"
- board text added: "60%"
- board text added: "80%"
- board text added: "A"
- board text added: "ANA"
- board text added: "BLU"
- board text added: "COM"
- board text added: "D-IN"
- board text added: "DC6.5-12V"
- board text added: "DIG"
- board text added: "DP"
- board text added: "GNDA"
- board text added: "GRN"
- board text added: "K"
- board text added: "RASPBERRY-Pi (Flip Insert)"
- board text added: "RED"
- board text added: "RPI"
- board text added: "SOURCE IND. LED"
- board text added: "X0"
- board text added: "X1"
- board text added: "X2"
- board text added: "XLR0+"
- board text added: "XLR0-"
- board text added: "XLR1+"
- board text added: "XLR1-"
- board text added: "XLR2+"
- board text added: "XLR2-"
- board text added: "XLR3+"
- board text added: "XLR3-"
- board text added: "XLR4+"
- board text added: "XLR4-"
- board text added: "XLR5+"
- board text added: "XLR5-"
- board text added: "XLR6+"
- board text added: "XLR6-"
- board text added: "XLR7+"
- board text added: "XLR7-"
- board text removed: "DIP"
- board text removed: "RASPBERRY-Pi"
- board text removed: "SOURCE IND, LED"
