File: SOURCES/kiCAD/DAC.sch (KiCad schematic (older format))
At the start: 186 parts, among them J16 MJ-519, J17 MJ-519, J20 MJ-519, J21 MJ-519, J24 Header6P, J25 Conn_01x06, J27 Conn_01x06, J28 Header6P, Q10 2SC3326, Q11 2SC3326, Q15 2SC3326, Q16 2SC3326, Q17 2SC3326, Q18 2SC3326, Q19 2SC3326, Q20 2SC3326, Q21 2SC3326, Q22 2SC3326, Q23 2SC3326, Q24 2SC3326, Q25 2SC3326, Q26 2SC3326, Q27 2SC3326, Q28 2SC3326, U14 PCM5102A, U16 PCM5102A, U17 PCM5102A, U18 PCM5102A, U20 OPA1632DR, U21 OPA1632DR, U22 OPA1632DR, U23 OPA1632DR, U24 OPA1632DR, U25 OPA1632DR, U26 OPA1632DR, U27 OPA1632DR

Commit message: Updated version0.2
Parts:
- J16, J17, J20, J21: JLPCB# NOP -> HAND
Changed lines of the file:
@@
 F 2 "MyJacks:MJ-519" H 15000 2775 50  0001 C CNN
 F 3 " ~" H 15000 2775 50  0001 C CNN
-F 4 "NOP" H 15000 2875 50  0001 C CNN "JLPCB#"
+F 4 "HAND" H 15000 2875 50  0001 C CNN "JLPCB#"
 	1    15000 2875
 	1    0    0    -1
@@
 F 2 "MyJacks:MJ-519" H 7675 6775 50  0001 C CNN
 F 3 " ~" H 7675 6775 50  0001 C CNN
-F 4 "NOP" H 7675 6875 50  0001 C CNN "JLPCB#"
+F 4 "HAND" H 7675 6875 50  0001 C CNN "JLPCB#"
 	1    7675 6875
 	1    0    0    -1
@@
 F 2 "MyJacks:MJ-519" H 14825 6650 50  0001 C CNN
 F 3 " ~" H 14825 6650 50  0001 C CNN
-F 4 "NOP" H 14825 6750 50  0001 C CNN "JLPCB#"
+F 4 "HAND" H 14825 6750 50  0001 C CNN "JLPCB#"
 	1    14825 6750
 	1    0    0    -1
@@
 F 2 "MyJacks:MJ-519" H 6850 2850 50  0001 C CNN
 F 3 " ~" H 6850 2850 50  0001 C CNN
-F 4 "NOP" H 6850 2950 50  0001 C CNN "JLPCB#"
+F 4 "HAND" H 6850 2950 50  0001 C CNN "JLPCB#"
 	1    6850 2950
 	1    0    0    -1

Commit message: Version0.2 Board. Reviced PCB design.
Parts:
- C114, C115, C116, C117, C96, C97, C98, C99: Description (none) -> use Audio-Grade or Film Cap (ie. PML, ECHU, etc..)
- J24, J28: value Header6P -> Conn_01x06; Description (none) -> for the XLR-Balanced Output; JLPCB# NOP -> NOP(BAL)
- J25, J27: Description (none) -> for the XLR-Balanced Output; JLPCB# NOP -> NOP(BAL)
- Q10, Q11, Q15, Q16, Q17, Q18, Q19, Q20, Q21, Q22, Q23, Q24, Q25, Q26, Q27, Q28: Description (none) -> alt. 2SC4213 or 2SD2704
Other:
- note added: "OUT-0\n(LEFT)\nOUT-1\n(RIGHT)"
- note added: "OUT-16\n(LEFT)\nOUT-17\n(RIGHT)\n(SUM-RIGHT)"
- note added: "OUT-32\n(LEFT)\nOUT-33\n(RIGHT)\n(SUM-LEFT)"
- note added: "OUT-40\n(LEFT)\nOUT-41\n(RIGHT)"
- note removed: "OUT-0\n\nOUT-1"
- note removed: "OUT-2\n\nOUT-3\n(LEFT)"
- note removed: "OUT-4\n\nOUT-5"
- note removed: "OUT-6\n\nOUT-7\n(RIGHT)"
Changed lines of the file:
@@
 Sheet 3 3
 Title "FreeDSP OCTAVIA DAC part"
-Date "2023-03-11"
-Rev "0.2"
+Date "2023-05-13"
+Rev "0.25"
 Comp ""
 Comment1 ""
@@
 F 3 "~" H 11000 2900 50  0001 C CNN
 F 4 "C408554" H 11000 2900 50  0001 C CNN "JLPCB#"
+F 5 "use Audio-Grade or Film Cap (ie. PML, ECHU, etc..)" H 11000 2900 50  0001 C CNN "Description"
 	1    11000 2900
 	1    0    0    1
@@
 F 3 "~" H 11250 2900 50  0001 C CNN
 F 4 "C408554" H 11250 2900 50  0001 C CNN "JLPCB#"
+F 5 "use Audio-Grade or Film Cap (ie. PML, ECHU, etc..)" H 11250 2900 50  0001 C CNN "Description"
 	1    11250 2900
 	1    0    0    1
@@
 F 3 "~" H 3550 6900 50  0001 C CNN
 F 4 "C408554" H 3550 6900 50  0001 C CNN "JLPCB#"
+F 5 "use Audio-Grade or Film Cap (ie. PML, ECHU, etc..)" H 3550 6900 50  0001 C CNN "Description"
 	1    3550 6900
 	1    0    0    1
@@
 F 3 "~" H 3800 6900 50  0001 C CNN
 F 4 "C408554" H 3800 6900 50  0001 C CNN "JLPCB#"
+F 5 "use Audio-Grade or Film Cap (ie. PML, ECHU, etc..)" H 3800 6900 50  0001 C CNN "Description"
 	1    3800 6900
 	1    0    0    1
@@
 F 3 "~" H 11200 6775 50  0001 C CNN
 F 4 "C408554" H 11200 6775 50  0001 C CNN "JLPCB#"
+F 5 "use Audio-Grade or Film Cap (ie. PML, ECHU, etc..)" H 11200 6775 50  0001 C CNN "Description"
 	1    11200 6775
 	1    0    0    1
@@
 F 3 "~" H 11450 6775 50  0001 C CNN
 F 4 "C408554" H 11450 6775 50  0001 C CNN "JLPCB#"
+F 5 "use Audio-Grade or Film Cap (ie. PML, ECHU, etc..)" H 11450 6775 50  0001 C CNN "Description"
 	1    11450 6775
 	1    0    0    1
@@
 F 2 "Connector_PinHeader_2.54mm:PinHeader_1x06_P2.54mm_Vertical" H 15025 4050 50  0001 C CNN
 F 3 "~" H 15025 4050 50  0001 C CNN
-F 4 "NOP" H 15025 4050 50  0001 C CNN "JLPCB#"
+F 4 "NOP(BAL)" H 15025 4050 50  0001 C CNN "JLPCB#"
+F 5 "for the XLR-Balanced Output" H 15025 4050 50  0001 C CNN "Description"
 	1    15025 4050
 	1    0    0    1
@@
 F 3 "~" H 13925 2800 50  0001 C CNN
 F 4 "C27829" H 13925 2800 50  0001 C CNN "JLPCB#"
+F 5 "alt. 2SC4213 or 2SD2704" H 13925 2800 50  0001 C CNN "Description"
 	1    13925 2800
 	1    0    0    1
@@
 F 3 "~" H 14025 3650 50  0001 C CNN
 F 4 "C27829" H 14025 3650 50  0001 C CNN "JLPCB#"
+F 5 "alt. 2SC4213 or 2SD2704" H 14025 3650 50  0001 C CNN "Description"
 	1    14025 3650
 	1    0    0    1
@@
 F 3 "~" H 13800 3400 50  0001 C CNN
 F 4 "C27829" H 13800 3400 50  0001 C CNN "JLPCB#"
+F 5 "alt. 2SC4213 or 2SD2704" H 13800 3400 50  0001 C CNN "Description"
 	1    13800 3400
 	1    0    0    1
@@
 F 2 "Connector_PinHeader_2.54mm:PinHeader_1x06_P2.54mm_Vertical" H 14850 7925 50  0001 C CNN
 F 3 "~" H 14850 7925 50  0001 C CNN
-F 4 "NOP" H 14850 7925 50  0001 C CNN "JLPCB#"
+F 4 "NOP(BAL)" H 14850 7925 50  0001 C CNN "JLPCB#"
+F 5 "for the XLR-Balanced Output" H 14850 7925 50  0001 C CNN "Description"
 	1    14850 7925
 	1    0    0    1
@@
 F 3 "~" H 13975 6675 50  0001 C CNN
 F 4 "C27829" H 13975 6675 50  0001 C CNN "JLPCB#"
+F 5 "alt. 2SC4213 or 2SD2704" H 13975 6675 50  0001 C CNN "Description"
 	1    13975 6675
 	1    0    0    1
@@
 F 3 "~" H 14075 7525 50  0001 C CNN
 F 4 "C27829" H 14075 7525 50  0001 C CNN "JLPCB#"
+F 5 "alt. 2SC4213 or 2SD2704" H 14075 7525 50  0001 C CNN "Description"
 	1    14075 7525
 	1    0    0    1
@@
 F 3 "~" H 13850 7275 50  0001 C CNN
 F 4 "C27829" H 13850 7275 50  0001 C CNN "JLPCB#"
+F 5 "alt. 2SC4213 or 2SD2704" H 13850 7275 50  0001 C CNN "Description"
 	1    13850 7275
 	1    0    0    1
@@
 Connection ~ 13275 7525
 Text Notes 14900 7875 0    63   ~ 0
-XLR4-POS\nXLR4-NEG\nAGND
+XLR6-POS\nXLR6-NEG\nAGND
 Connection ~ 11200 6525
 Connection ~ 11450 6425
@@
 P 7700 8050
 F 0 "J28" H 7625 8350 50  0000 L CNN
-F 1 "Header6P" H 7625 8425 50  0000 L CNN
+F 1 "Conn_01x06" H 7625 8425 50  0000 L CNN
 F 2 "Connector_PinHeader_2.54mm:PinHeader_1x06_P2.54mm_Vertical" H 7700 8050 50  0001 C CNN
 F 3 "~" H 7700 8050 50  0001 C CNN
-F 4 "NOP" H 7700 8050 50  0001 C CNN "JLPCB#"
+F 4 "NOP(BAL)" H 7700 8050 50  0001 C CNN "JLPCB#"
+F 5 "for the XLR-Balanced Output" H 7700 8050 50  0001 C CNN "Description"
 	1    7700 8050
 	1    0    0    1
@@
 F 3 "~" H 6800 6800 50  0001 C CNN
 F 4 "C27829" H 6800 6800 50  0001 C CNN "JLPCB#"
+F 5 "alt. 2SC4213 or 2SD2704" H 6800 6800 50  0001 C CNN "Description"
 	1    6800 6800
 	1    0    0    1
@@
 F 3 "~" H 6900 7650 50  0001 C CNN
 F 4 "C27829" H 6900 7650 50  0001 C CNN "JLPCB#"
+F 5 "alt. 2SC4213 or 2SD2704" H 6900 7650 50  0001 C CNN "Description"
 	1    6900 7650
 	1    0    0    1
@@
 F 3 "~" H 6675 7400 50  0001 C CNN
 F 4 "C27829" H 6675 7400 50  0001 C CNN "JLPCB#"
+F 5 "alt. 2SC4213 or 2SD2704" H 6675 7400 50  0001 C CNN "Description"
 	1    6675 7400
 	1    0    0    1
@@
 Connection ~ 6100 7650
 Text Notes 7750 8000 0    63   ~ 0
-XLR6-POS\nXLR6-NEG\nAGND
+XLR2-POS\nXLR2-NEG\nAGND
 Connection ~ 3550 6650
 Connection ~ 3800 6550
@@
 MUTE
 Text Notes 15075 4300 0    63   ~ 0
-XLR3-POS\nXLR3-NEG\nAGND
-Text Notes 14900 8175 0    63   ~ 0
 XLR5-POS\nXLR5-NEG\nAGND
-Text Notes 7750 8300 0    63   ~ 0
+Text Notes 14900 8175 0    63   ~ 0
 XLR7-POS\nXLR7-NEG\nAGND
+Text Notes 7750 8300 0    63   ~ 0
+XLR3-POS\nXLR3-NEG\nAGND
 Connection ~ 14125 2575
 Connection ~ 13125 3200
@@
 	9200 8125 13275 8125
 Text Notes 15075 4000 0    63   ~ 0
-XLR2-POS\nXLR2-NEG\nAGND
+XLR4-POS\nXLR4-NEG\nAGND
 Wire Wire Line
 	13825 2075 12825 2075
@@
 F 3 "~" H 13725 2350 50  0001 C CNN
 F 4 "C27829" H 13725 2350 50  0001 C CNN "JLPCB#"
+F 5 "alt. 2SC4213 or 2SD2704" H 13725 2350 50  0001 C CNN "Description"
 	1    13725 2350
 	1    0    0    1
@@
 F 3 "~" H 5975 3475 50  0001 C CNN
 F 4 "C27829" H 5975 3475 50  0001 C CNN "JLPCB#"
+F 5 "alt. 2SC4213 or 2SD2704" H 5975 3475 50  0001 C CNN "Description"
 	1    5975 3475
 	1    0    0    1
@@
 F 3 "~" H 6200 3725 50  0001 C CNN
 F 4 "C27829" H 6200 3725 50  0001 C CNN "JLPCB#"
+F 5 "alt. 2SC4213 or 2SD2704" H 6200 3725 50  0001 C CNN "Description"
 	1    6200 3725
 	1    0    0    1
@@
 F 3 "~" H 5900 2425 50  0001 C CNN
 F 4 "C27829" H 5900 2425 50  0001 C CNN "JLPCB#"
+F 5 "alt. 2SC4213 or 2SD2704" H 5900 2425 50  0001 C CNN "Description"
 	1    5900 2425
 	1    0    0    1
@@
 F 3 "~" H 6100 2875 50  0001 C CNN
 F 4 "C27829" H 6100 2875 50  0001 C CNN "JLPCB#"
+F 5 "alt. 2SC4213 or 2SD2704" H 6100 2875 50  0001 C CNN "Description"
 	1    6100 2875
 	1    0    0    1
@@
 P 6875 4125
 F 0 "J24" H 6800 4500 50  0000 L CNN
-F 1 "Header6P" H 6775 4425 50  0000 L CNN
+F 1 "Conn_01x06" H 6775 4425 50  0000 L CNN
 F 2 "Connector_PinHeader_2.54mm:PinHeader_1x06_P2.54mm_Vertical" H 6875 4125 50  0001 C CNN
 F 3 "~" H 6875 4125 50  0001 C CNN
-F 4 "NOP" H 6875 4125 50  0001 C CNN "JLPCB#"
+F 4 "NOP(BAL)" H 6875 4125 50  0001 C CNN "JLPCB#"
+F 5 "for the XLR-Balanced Output" H 6875 4125 50  0001 C CNN "Description"
 	1    6875 4125
 	1    0    0    1
@@
 U 1 1 65D99AA6
 P 6850 2950
-F 0 "J17" H 6800 3250 50  0000 L CNN
-F 1 "MJ-519" H 6800 3175 50  0000 L CNN
+F 0 "J17" H 6775 3325 50  0000 L CNN
+F 1 "MJ-519" H 6725 3250 50  0000 L CNN
 F 2 "MyJacks:MJ-519" H 6850 2850 50  0001 C CNN
 F 3 " ~" H 6850 2850 50  0001 C CNN
@@
 F 3 "~" H 3575 2975 50  0001 C CNN
 F 4 "C408554" H 3575 2975 50  0001 C CNN "JLPCB#"
+F 5 "use Audio-Grade or Film Cap (ie. PML, ECHU, etc..)" H 3575 2975 50  0001 C CNN "Description"
 	1    3575 2975
 	1    0    0    1
@@
 F 3 "~" H 3325 2975 50  0001 C CNN
 F 4 "C408554" H 3325 2975 50  0001 C CNN "JLPCB#"
+F 5 "use Audio-Grade or Film Cap (ie. PML, ECHU, etc..)" H 3325 2975 50  0001 C CNN "Description"
 	1    3325 2975
 	1    0    0    1
@@
 DAC2_R
 Text Notes 6950 3100 0    63   ~ 0
-OUT-0\n\nOUT-1
-Text Notes 15100 3125 0    63   ~ 0
-OUT-2\n\nOUT-3\n(LEFT)
-Text Notes 14925 6900 0    63   ~ 0
-OUT-4\n\nOUT-5
-Text Notes 7775 7125 0    63   ~ 0
-OUT-6\n\nOUT-7\n(RIGHT)
+OUT-0\n(LEFT)\nOUT-1\n(RIGHT)
+Text Notes 15100 3175 0    63   ~ 0
+OUT-32\n(LEFT)\nOUT-33\n(RIGHT)\n(SUM-LEFT)
+Text Notes 14925 6975 0    63   ~ 0
+OUT-40\n(LEFT)\nOUT-41\n(RIGHT)
+Text Notes 7775 7200 0    63   ~ 0
+OUT-16\n(LEFT)\nOUT-17\n(RIGHT)\n(SUM-RIGHT)
 Wire Wire Line
 	6400 4225 6675 4225
@@
 F 3 "~" H 13775 6225 50  0001 C CNN
 F 4 "C27829" H 13775 6225 50  0001 C CNN "JLPCB#"
+F 5 "alt. 2SC4213 or 2SD2704" H 13775 6225 50  0001 C CNN "Description"
 	1    13775 6225
 	1    0    0    1
@@
 F 3 "~" H 6600 6350 50  0001 C CNN
 F 4 "C27829" H 6600 6350 50  0001 C CNN "JLPCB#"
+F 5 "alt. 2SC4213 or 2SD2704" H 6600 6350 50  0001 C CNN "Description"
 	1    6600 6350
 	1    0    0    1

Commit message: Fixed wrong L/R Connection of RCA Jack
Connections:
- net at J24.5 (Pin_5), Q16.2 (E), R137.2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: now also J17.2 (IN2); no longer J17.1 (IN1)
- net at J24.2 (Pin_2), Q18.2 (E), R139.2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: now also J17.1 (IN1); no longer J17.2 (IN2)
- net at J25.5 (Pin_5), Q19.2 (E), R148.2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: now also J21.2 (IN2); no longer J21.1 (IN1)
- net at J25.2 (Pin_2), Q20.2 (E), R150.2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: now also J21.1 (IN1); no longer J21.2 (IN2)
- net at J27.5 (Pin_5), Q23.2 (E), R178.2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: now also J20.2 (IN2); no longer J20.1 (IN1)
- net at J27.2 (Pin_2), Q24.2 (E), R180.2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: now also J20.1 (IN1); no longer J20.2 (IN2)
- net at J28.5 (Pin_5), Q27.2 (E), R189.2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: now also J16.2 (IN2); no longer J16.1 (IN1)
- net at J28.2 (Pin_2), Q28.2 (E), R191.2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: now also J16.1 (IN1); no longer J16.2 (IN2)
Other:
- note added: "H=UnMute\nL=SoftMute"
- note added: "OUT-0\n(RIGHT)\nOUT-1\n(LEFT)"
- note added: "OUT-16\n(RIGHT)\nOUT-17\n(LEFT)\n(SUM-RIGHT)"
- note added: "OUT-32\n(RIGHT)\nOUT-33\n(LEFT)\n(SUM-LEFT)"
- note added: "OUT-40\n(RIGHT)\nOUT-41\n(LEFT)"
- note removed: "OUT-0\n(LEFT)\nOUT-1\n(RIGHT)"
- note removed: "OUT-16\n(LEFT)\nOUT-17\n(RIGHT)\n(SUM-RIGHT)"
- note removed: "OUT-32\n(LEFT)\nOUT-33\n(RIGHT)\n(SUM-LEFT)"
- note removed: "OUT-40\n(LEFT)\nOUT-41\n(RIGHT)"
Changed lines of the file:
@@
 Sheet 3 3
 Title "FreeDSP OCTAVIA DAC part"
-Date "2023-05-13"
-Rev "0.25"
+Date "2023-05-25"
+Rev "0.26"
 Comp ""
 Comment1 ""
@@
 $EndComp
 Wire Wire Line
-	14800 2775 14125 2775
-Connection ~ 14125 2775
-Wire Wire Line
-	14125 2775 14125 3125
-Wire Wire Line
-	14800 2975 14225 2975
-Wire Wire Line
-	14225 2975 14225 3425
-Wire Wire Line
 	14825 4150 14225 4150
 Wire Wire Line
@@
 Wire Wire Line
 	14025 2575 14125 2575
-Wire Wire Line
-	14125 2575 14125 2775
 $Comp
 L fdsp_power:GNDA #PWR0154
@@
 	1    0    0    -1
 $EndComp
-Connection ~ 14175 6650
-Wire Wire Line
-	14175 6650 14175 7000
-Wire Wire Line
-	14275 6850 14275 7300
 Wire Wire Line
 	12875 8025 14275 8025
@@
 	14075 6450 14175 6450
 Connection ~ 14175 6450
-Wire Wire Line
-	14175 6450 14175 6650
 $Comp
 L fdsp_power:GNDA #PWR0175
@@
 	7450 8250 7450 8275
 Wire Wire Line
-	7475 6775 7000 6775
-Connection ~ 7000 6775
-Wire Wire Line
-	7000 6775 7000 7125
-Wire Wire Line
-	7475 6975 7100 6975
-Wire Wire Line
-	7100 6975 7100 7425
-Wire Wire Line
 	6000 8050 6000 7325
 Wire Wire Line
@@
 	6900 6575 7000 6575
 Connection ~ 7000 6575
-Wire Wire Line
-	7000 6575 7000 6775
 $Comp
 L fdsp_power:GNDA #PWR0179
@@
 	1    0    0    -1
 $EndComp
-Wire Wire Line
-	6300 2650 6300 2850
 Connection ~ 6300 2650
 Wire Wire Line
@@
 	5000 4225 6400 4225
 Wire Wire Line
-	6400 3050 6400 3500
-Wire Wire Line
-	6650 3050 6400 3050
-Wire Wire Line
-	6300 2850 6300 3200
-Connection ~ 6300 2850
-Wire Wire Line
-	6650 2850 6300 2850
-Wire Wire Line
 	6625 4325 6625 4350
 $Comp
@@
 DAC2_R
 Text Notes 6950 3100 0    63   ~ 0
-OUT-0\n(LEFT)\nOUT-1\n(RIGHT)
+OUT-0\n(RIGHT)\nOUT-1\n(LEFT)
 Text Notes 15100 3175 0    63   ~ 0
-OUT-32\n(LEFT)\nOUT-33\n(RIGHT)\n(SUM-LEFT)
+OUT-32\n(RIGHT)\nOUT-33\n(LEFT)\n(SUM-LEFT)
 Text Notes 14925 6975 0    63   ~ 0
-OUT-40\n(LEFT)\nOUT-41\n(RIGHT)
+OUT-40\n(RIGHT)\nOUT-41\n(LEFT)
 Text Notes 7775 7200 0    63   ~ 0
-OUT-16\n(LEFT)\nOUT-17\n(RIGHT)\n(SUM-RIGHT)
+OUT-16\n(RIGHT)\nOUT-17\n(LEFT)\n(SUM-RIGHT)
 Wire Wire Line
 	6400 4225 6675 4225
@@
 Connection ~ 14600 8125
 Wire Wire Line
-	14175 6650 14625 6650
-Wire Wire Line
-	14275 6850 14625 6850
-Wire Wire Line
 	14550 7625 14550 5950
 Wire Wire Line
@@
 Wire Wire Line
 	3075 3425 3075 3500
+Text Notes 775  3400 0    50   ~ 0
+H=UnMute\nL=SoftMute
+Text Notes 8400 3350 0    50   ~ 0
+H=UnMute\nL=SoftMute
+Text Notes 8625 7200 0    50   ~ 0
+H=UnMute\nL=SoftMute
+Text Notes 975  7325 0    50   ~ 0
+H=UnMute\nL=SoftMute
+Wire Wire Line
+	6300 2650 6300 3050
+Wire Wire Line
+	6650 2850 6400 2850
+Wire Wire Line
+	6400 2850 6400 3500
+Wire Wire Line
+	6650 3050 6300 3050
+Connection ~ 6300 3050
+Wire Wire Line
+	6300 3050 6300 3200
+Wire Wire Line
+	14125 2575 14125 2975
+Wire Wire Line
+	14800 2775 14225 2775
+Wire Wire Line
+	14225 2775 14225 3425
+Wire Wire Line
+	14800 2975 14125 2975
+Connection ~ 14125 2975
+Wire Wire Line
+	14125 2975 14125 3125
+Wire Wire Line
+	14175 6450 14175 6850
+Wire Wire Line
+	14625 6650 14275 6650
+Wire Wire Line
+	14275 6650 14275 7300
+Wire Wire Line
+	14625 6850 14175 6850
+Connection ~ 14175 6850
+Wire Wire Line
+	14175 6850 14175 7000
+Wire Wire Line
+	7000 6575 7000 6975
+Wire Wire Line
+	7475 6775 7100 6775
+Wire Wire Line
+	7100 6775 7100 7425
+Wire Wire Line
+	7475 6975 7000 6975
+Connection ~ 7000 6975
+Wire Wire Line
+	7000 6975 7000 7125
 $EndSCHEMATC

Commit message: New Output Driver with Enhanced 4 Layer PCB
Parts:
- removed R136, R147, R149, R179, R188, R190: 4.7k, Resistor_SMD:R_0603_1608Metric, symbol Device:R
- removed R143: NOP, Resistor_SMD:R_0603_1608Metric, symbol Device:R
- removed R157, R158, R199, R200: 330R, Resistor_SMD:R_0603_1608Metric, symbol Device:R
- removed R197: 0R, Resistor_SMD:R_0805_2012Metric_Pad1.20x1.40mm_HandSolder, symbol Device:R
- added C144, C146, C150, C151, C157, C158, C160, C161: 470pF(C0G), Capacitor_SMD:C_0805_2012Metric_Pad1.18x1.45mm_HandSolder, symbol Device:C_Small
- added C145, C149, C154, C159: 0.1uF, Capacitor_SMD:C_0603_1608Metric, symbol Device:C_Small
- added C147, C148, C152, C153, C155, C156, C162, C163: NOP, Capacitor_SMD:C_0805_2012Metric_Pad1.18x1.45mm_HandSolder, symbol Device:C_Small
- added R52: 10R, Resistor_SMD:R_0603_1608Metric, symbol Device:R
- added R53: 0R, Resistor_SMD:R_0603_1608Metric, symbol Device:R
- C114, C115, C116, C117, C96, C97, C98, C99: value 1nF(C0G) -> 10nF(C0G); Description use Audio-Grade or Film Cap (ie. PML, ECHU, etc..) -> se Audio-Grade or Film Cap (ie. PML, ECHU, etc..); JLPCB# C408554 -> C342877
- R132, R134, R140, R142, R173, R175, R181, R183: value 4.7k -> 1.1k; JLPCB# C23162 -> C22764
- R133, R135, R137, R139, R141, R146, R148, R150, R174, R176, R178, R180, R182, R187, R189, R191: value 4.7k -> 2.2k; JLPCB# C23162 -> C4190
- R138: value 4.7k -> 0R; JLPCB# C23162 -> C21189
- R144, R145, R184, R185: value NOP -> 10R; JLPCB# NOP -> C22859
- R151, R153: value 330R -> 10R; JLPCB# C23138 -> C22859
- R152, R154, R159, R160, R192, R193, R194, R195, R198, R201: value 330R -> 220R; JLPCB# C23138 -> C22962
- R155, R156, R161, R162, R203, R204: value 0R -> 220R; footprint Resistor_SMD:R_0805_2012Metric_Pad1.20x1.40mm_HandSolder -> Resistor_SMD:R_0603_1608Metric; JLPCB# C17477 -> C22962
- R163, R164, R165, R166, R167, R168, R169, R170, R202, R205, R206, R207, R208, R209, R210, R211: footprint Resistor_SMD:R_0805_2012Metric_Pad1.20x1.40mm_HandSolder -> Resistor_SMD:R_0603_1608Metric; JLPCB# C17414 -> C25804
- R171, R172, R212, R213: value 100R -> NOP; footprint Resistor_SMD:R_0805_2012Metric_Pad1.20x1.40mm_HandSolder -> Resistor_SMD:R_0603_1608Metric; JLPCB# C17408 -> NOP
- R177: value 4.7k -> 10R; JLPCB# C23162 -> C22859
- R186: value NOP -> 0R; JLPCB# NOP -> C21189
- R196: footprint Resistor_SMD:R_0805_2012Metric_Pad1.20x1.40mm_HandSolder -> Resistor_SMD:R_0603_1608Metric; JLPCB# C17477 -> C21189
Connections:
- net DAC0_L: now also R133.1; no longer R132.2
- net DAC0_R: now also R135.2; no longer R134.2, R145.2
- net DAC2_L: now also C98.2, R122.1, R141.1; no longer C116.2, R126.1, R173.2, R184.2
- net DAC2_R: now also C96.2, R123.1, R146.2; no longer C114.2, R127.1, R175.2, R186.2
- net GNDA: now also R132.2, R134.2, R138.1, R140.2, R142.2, R144.2, R151.1, R173.2, R175.2, R177.2, R181.2, R183.2, R184.2, R186.2, R196.1, C145.1, C149.2, C154.1, C159.1, R53.1; no longer J24.1 (Pin_1), J24.4 (Pin_4), J25.1 (Pin_1), J25.4 (Pin_4), J27.1 (Pin_1), J27.4 (Pin_4), J28.1 (Pin_1), J28.4 (Pin_4), Q10.3 (C), Q11.3 (C), Q15.3 (C), Q16.3 (C), Q17.3 (C), Q18.3 (C), Q19.3 (C), Q20.3 (C), Q21.3 (C), Q22.3 (C), Q23.3 (C), Q24.3 (C), Q25.3 (C), Q26.3 (C), Q27.3 (C), Q28.3 (C), R133.1, R135.1, R141.1, R146.2, R171.2, R172.2, R174.1, R176.1, R182.1, R187.1, R212.2, R213.2, U20.2 (VCOM), U21.2 (VCOM), U22.2 (VCOM), U23.2 (VCOM), U24.2 (VCOM), U25.2 (VCOM), U26.2 (VCOM), U27.2 (VCOM)
- net at R132.1, U20.1 (IN-): now also C155.1
- net at R151.2: now also R153.1, U20.2 (VCOM), U21.2 (VCOM), C154.2; no longer U20.4 (OUT+)
- net at R152.1, U20.5 (OUT-): now also R137.2, C157.1
- net at R133.2, R137.1, U20.8 (IN+): now also C157.2
- net OUT1_P: now reaches J24.6 (Pin_6), Q10.2 (E)
- net OUT1_P: now also J17.2 (IN2), R155.2; no longer R151.1, R155.1
- net OUT0_N: now reaches J24.5 (Pin_5), Q16.2 (E), R152.2
- net OUT0_N: no longer J17.2 (IN2), R137.2
- net at R134.1, U21.1 (IN-): now also C156.1; no longer R138.2
- net at U21.4 (OUT+): now also R156.2, C156.2; no longer R153.2
- net at R154.1, U21.5 (OUT-): now also R139.2, C158.1
- net at R139.1, U21.8 (IN+): now also R135.1, C158.2; no longer R135.2
- net OUT1_N: now reaches J24.2 (Pin_2), Q18.2 (E), R154.2
- net OUT1_N: no longer J17.1 (IN1), R139.2
- net at R140.1, U24.1 (IN-): now also C153.1
- net at U24.4 (OUT+): now also R161.1, C153.2
- net at U24.5 (OUT-): now also R148.2, R160.1, C150.1
- net at R141.2, R148.1, U24.8 (IN+): now also C150.2
- net OUT32_P: now reaches J25.6 (Pin_6), Q15.2 (E)
- net OUT32_P: now also J21.2 (IN2), R161.2; no longer R161.1
- net OUT32_N: now reaches J25.5 (Pin_5), Q19.2 (E)
- net OUT32_N: now also R160.2; no longer J21.2 (IN2), R148.2
- net at R142.1, U25.1 (IN-): now also C152.1
- net at U25.4 (OUT+): now also R162.2, C152.2; no longer R159.2
- net at U25.5 (OUT-): now also R150.2, R159.1, C151.1; no longer R160.1
- net at R146.1, R150.1, U25.8 (IN+): now also C151.2; no longer R144.1, R145.1
- net at R173.1, U26.1 (IN-): now also C148.1; no longer R177.2
- net at U26.4 (OUT+): now also R192.1, C148.2; no longer R192.2
- net at R193.1, U26.5 (OUT-): now also R178.2, C144.1
- net at R174.2, R178.1, U26.8 (IN+): now also C144.2
- net OUT40_N: now reaches J27.5 (Pin_5), Q23.2 (E), R193.2
- net OUT40_N: no longer J20.2 (IN2), R178.2
- net DIFF_GND3: now reaches J20.3 (EXT), R212.1
- net DIFF_GND3: now also R52.2; no longer Q22.2 (E), R196.2
- net at R175.1, U27.1 (IN-): now also C147.1
- net at R194.2, U27.4 (OUT+): now also C147.2
- net at R195.1, U27.5 (OUT-): now also R180.2, C146.1
- net at R176.2, R180.1, U27.8 (IN+): now also C146.2
- net OUT41_P: now reaches J27.3 (Pin_3), R194.1
- net OUT41_P: now also J20.1 (IN1), Q22.2 (E)
- net OUT41_N: now reaches J27.2 (Pin_2), Q24.2 (E), R195.2
- net OUT41_N: no longer J20.1 (IN1), R180.2
- net DAC1_L: now reaches C117.2, R128.1
- net DAC1_L: now also R182.1; no longer R181.2, R185.2
- net DAC1_R: now reaches C115.2, R129.1
- net DAC1_R: now also R187.1; no longer R183.2
- net OUT17_N: now reaches J28.2 (Pin_2), Q28.2 (E), R201.2
- net OUT17_N: no longer J16.1 (IN1), R191.2
- net OUT16_N: now reaches J28.5 (Pin_5), Q27.2 (E)
- net OUT16_N: now also R198.2; no longer J16.2 (IN2), R189.2
- net at R181.1, U22.1 (IN-): now also C163.1
- net at U22.4 (OUT+): now also R203.1, C163.2; no longer R198.2
- net at U22.5 (OUT-): now also R189.2, R198.1, C160.1
- net at R182.2, R189.1, U22.8 (IN+): now also C160.2
- net OUT16_P: now reaches J28.6 (Pin_6), Q25.2 (E)
- net OUT16_P: now also J16.2 (IN2), R203.2; no longer R198.1, R203.1
- net at R183.1, U23.1 (IN-): now also C162.1; no longer R184.1
- net at U23.4 (OUT+): now also R204.2, C162.2
- net at R201.1, U23.5 (OUT-): now also R191.2, C161.1
- net at R187.2, R191.1, U23.8 (IN+): now also C161.2; no longer R185.1, R186.1
- net OUT17_P: now reaches J28.3 (Pin_3)
- net OUT17_P: now also J16.1 (IN1), Q26.2 (E), R204.1; no longer R204.2
- new net: C155.2, R155.1, U20.4 (OUT+)
- new net: C149.1, R144.1, R145.2, U24.2 (VCOM), U25.2 (VCOM)
- new net: C145.2, R177.1, R52.1, U26.2 (VCOM), U27.2 (VCOM)
- new net: C159.2, R184.1, R185.2, U22.2 (VCOM), U23.2 (VCOM)
- new net DAC3_L: C116.2, R126.1, R174.1
- new net DAC3_R: C114.2, R127.1, R176.1
- new net DIFF_GND0: J17.3 (EXT), R153.2, R171.1
- new net DIFF_GND1: J16.3 (EXT), R185.1, R213.1
- new net DIFF_GND2: J21.3 (EXT), R145.1, R172.2
- new net MUTE_GND0: J24.1 (Pin_1), J24.4 (Pin_4), Q10.3 (C), Q11.3 (C), Q16.3 (C), Q18.3 (C), R138.2, R171.2
- new net MUTE_GND1: J28.1 (Pin_1), J28.4 (Pin_4), Q25.3 (C), Q26.3 (C), Q27.3 (C), Q28.3 (C), R186.1, R213.2
- new net MUTE_GND2: J25.1 (Pin_1), J25.4 (Pin_4), Q15.3 (C), Q17.3 (C), Q19.3 (C), Q20.3 (C), R172.1, R53.2
- new net MUTE_GND3: J27.1 (Pin_1), J27.4 (Pin_4), Q21.3 (C), Q22.3 (C), Q23.3 (C), Q24.3 (C), R196.2, R212.2
- new net OUT0_P: J17.1 (IN1), J24.3 (Pin_3), Q11.2 (E), R156.1
- new net OUT33_N: J25.2 (Pin_2), Q20.2 (E), R159.2
- new net OUT33_P: J21.1 (IN1), J25.3 (Pin_3), Q17.2 (E), R162.1
- new net OUT40_P: J20.2 (IN2), J27.6 (Pin_6), Q21.2 (E), R192.2
Other:
- note added: "DO NOT CONNECT XLR AND RCA SIMULTINIEOUSULY\n(XLR OUTPUT WILL NOT BE BALANCED)"
- note added: "OUT-16\n(RIGHT)\nOUT-17\n(LEFT)"
- note added: "OUT-32\n(RIGHT)\nOUT-33\n(LEFT)"
- note added: "REMOVE;\n U26, U27, Q21, Q22, R202, R205, R173, R175, R194, R192, C145\n\nCHANGE:\n (to 0R) R174, R178, R193, R176, R180, R195, R177, R52\n\nJUMPER:\n Between J27 pin6-pin5, Between J27 pin2-pin3"
- note added: "To Create FreeDSP OVTAVIA Basic version Example"
- note added: "XLR/RCA RCA ONLY\n\nR171 NOPOP 0R \n\nR138 0R NOPOP"
- note added: "XLR/RCA RCA ONLY\n\nR172 NOPOP 0R \n\n R53 0R NOPOP"
- note added: "XLR/RCA RCA ONLY\n\nR212 NOPOP 0R \n\nR196 0R NOPOP"
- note added: "XLR/RCA RCA ONLY\n\nR213 NOPOP 0R \n\nR186 0R NOPOP"
- note added: "XLR0-POS\nXLR0-NEG\nGND0"
- note added: "XLR1-POS\nXLR1-NEG\nGND1"
- note added: "XLR2-POS\nXLR2-NEG\nGND2"
- note added: "XLR3-POS\nXLR3-NEG\nGND3"
- note added: "XLR4-POS\nXLR4-NEG\nGND4"
- note added: "XLR5-POS\nXLR5-NEG\nGND5"
- note added: "XLR6-POS\nXLR6-NEG\nGND6"
- note added: "XLR7-POS\nXLR7-NEG\nGND7"
- note removed: "CHANE (to Zero Ohm): R181, R188, R183, R190, R213"
- note removed: "CHANGE:\n(to 10k) R183, R184, R185, R186\n(to MJ-518 or Butique Jacks) J16"
- note removed: "FreeDSP OVTAVIA (Extend S/N 6dB stereo version)"
- note removed: "FreeDSP OVTAVIA (Extend S/N 6dB version)"
- note removed: "JUMPER(Between): J28 pin2-Pin3, pin5-pin6"
- note removed: "NOT POPULATE : U22, U23, R182, R189, R187, R191, R199, R201, R203, R209, Q26, R208, Q25, R204, R198, R200"
- note removed: "NOT POPULATE: J16, R213, R203"
- note removed: "NOT POPULATE: Q25, R208 (if you want)"
- note removed: "NOT POPULATE: \nU26, U21, Q23, Q22, Q24, J20, J27, R202, R206, R205, R207, R212, R196, R197, R192, R193, R194, R195, \nR177, R173, R174, R178, R175, R179, R176, R180, U22, Q25, Q27, R208, R210, R209, R210, R203, R198, R199, R188, R181, R189, R182"
- note removed: "OUT-16\n(RIGHT)\nOUT-17\n(LEFT)\n(SUM-RIGHT)"
- note removed: "OUT-32\n(RIGHT)\nOUT-33\n(LEFT)\n(SUM-LEFT)"
- note removed: "XLR0-POS\nXLR0-NEG\nAGND"
- note removed: "XLR1-POS\nXLR1-NEG\nAGND"
- note removed: "XLR2-POS\nXLR2-NEG\nAGND"
- note removed: "XLR3-POS\nXLR3-NEG\nAGND"
- note removed: "XLR4-POS\nXLR4-NEG\nAGND"
- note removed: "XLR5-POS\nXLR5-NEG\nAGND"
- note removed: "XLR6-POS\nXLR6-NEG\nAGND"
- note removed: "XLR7-POS\nXLR7-NEG\nAGND"
- moved on the sheet: C114, C116, C117, C123, C124, C125, C126, C127, C128, C129, C130, C131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
