File: SOURCES/kiCAD/DAC.sch (KiCad schematic (older format))
At the start: 196 parts, among them J16 MJ-519, J17 MJ-519, J20 MJ-519, J21 MJ-519, J24 Conn_01x06, J25 Conn_01x06, J27 Conn_01x06, J28 Conn_01x06, Q10 2SC3326, Q11 2SC3326, Q15 2SC3326, Q16 2SC3326, Q17 2SC3326, Q18 2SC3326, Q19 2SC3326, Q20 2SC3326, Q21 2SC3326, Q22 2SC3326, Q23 2SC3326, Q24 2SC3326, Q25 2SC3326, Q26 2SC3326, Q27 2SC3326, Q28 2SC3326, U14 PCM5102A, U16 PCM5102A, U17 PCM5102A, U18 PCM5102A, U20 OPA1632DR, U21 OPA1632DR, U22 OPA1632DR, U23 OPA1632DR, U24 OPA1632DR, U25 OPA1632DR, U26 OPA1632DR, U27 OPA1632DR

Commit message: Released for everyone, ready to build.
Parts:
- FB10, FB11, FB12, FB5, FB6, FB7, FB8, FB9: Description (none) -> Filter for DAC Power Rail
- J16, J17, J20, J21: value MJ-519 -> RCJ-2223; footprint MyJacks:MJ-519 -> MyJacks:RCJ-2223; Description Vertical Stereo RCA-pin Jack (Upper=Left, Lower=Right) RCJ-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 -> Vertical Stereo RCA-pin Jack (Upper=Right, Lower=Left) RCJ-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
- R138: Description (none) -> Move to R171 when never use of XLR
- R171, R172, R212, R213: Description (none) -> Nount Zero-R when Non-Lifting GND RCA-pin Output
- R186: Description (none) -> Move to R213 when never use of XLR
- R196: Description (none) -> Move to R212 when never use of XLR
- R53: Description (none) -> Move to R172 when never use of XLR
Connections:
- net OUT0_P: now also J17.2 (IN2), J24.6 (Pin_6), Q10.2 (E), R155.2; no longer J17.1 (IN1), J24.3 (Pin_3), Q11.2 (E), R156.1
- net OUT1_P: now also J17.1 (IN1), J24.3 (Pin_3), Q11.2 (E), R156.1; no longer J17.2 (IN2), J24.6 (Pin_6), Q10.2 (E), R155.2
Other:
- note added: "CUI"
- note added: "OUT-17\n(RIGHT)\nOUT-16\n(LEFT)"
- note added: "OUT-1\n(RIGHT)\nOUT-0\n(LEFT)\n"
- note added: "OUT-33\n(RIGHT)\nOUT-32\n(LEFT)\n"
- note added: "OUT-41\n(RIGHT)\nOUT-40\n(LEFT)\n"
- note removed: "CUI RCJ-2232(2233)"
- note removed: "OUT-0\n(RIGHT)\nOUT-1\n(LEFT)"
- note removed: "OUT-16\n(RIGHT)\nOUT-17\n(LEFT)"
- note removed: "OUT-32\n(RIGHT)\nOUT-33\n(LEFT)"
- note removed: "OUT-40\n(RIGHT)\nOUT-41\n(LEFT)"
Changed lines of the file:
@@
 Sheet 3 3
 Title "FreeDSP OCTAVIA DAC part"
-Date "2023-08-27"
-Rev "0.33"
+Date "2023-09-30"
+Rev "1.00"
 Comp ""
 Comment1 ""
@@
 P 14900 2650
 F 0 "J21" H 14850 2875 50  0000 L CNN
-F 1 "MJ-519" H 14850 2950 50  0000 L CNN
-F 2 "MyJacks:MJ-519" H 14900 2550 50  0001 C CNN
+F 1 "RCJ-2223" H 14850 2950 50  0000 L CNN
+F 2 "MyJacks:RCJ-2223" H 14900 2550 50  0001 C CNN
 F 3 " ~" H 14900 2550 50  0001 C CNN
 F 4 "HAND" H 14900 2650 50  0001 C CNN "JLPCB#"
-F 5 "Vertical Stereo RCA-pin Jack (Upper=Left, Lower=Right) RCJ-2232,RCJ-2233" H 14900 2650 50  0001 C CNN "Description"
+F 5 "Vertical Stereo RCA-pin Jack (Upper=Right, Lower=Left) RCJ-2223" H 14900 2650 50  0001 C CNN "Description"
 	1    14900 2650
 	1    0    0    -1
@@
 P 7750 6800
 F 0 "J16" H 7700 7025 50  0000 L CNN
-F 1 "MJ-519" H 7525 7150 50  0000 L CNN
-F 2 "MyJacks:MJ-519" H 7750 6700 50  0001 C CNN
+F 1 "RCJ-2223" H 7525 7150 50  0000 L CNN
+F 2 "MyJacks:RCJ-2223" H 7750 6700 50  0001 C CNN
 F 3 " ~" H 7750 6700 50  0001 C CNN
 F 4 "HAND" H 7750 6800 50  0001 C CNN "JLPCB#"
-F 5 "Vertical Stereo RCA-pin Jack (Upper=Left, Lower=Right) RCJ-2232,RCJ-2233" H 7750 6800 50  0001 C CNN "Description"
+F 5 "Vertical Stereo RCA-pin Jack (Upper=Right, Lower=Left) RCJ-2223" H 7750 6800 50  0001 C CNN "Description"
 	1    7750 6800
 	1    0    0    -1
@@
 P 15100 6675
 F 0 "J20" H 15050 6900 50  0000 L CNN
-F 1 "MJ-519" H 15050 6975 50  0000 L CNN
-F 2 "MyJacks:MJ-519" H 15100 6575 50  0001 C CNN
+F 1 "RCJ-2223" H 15050 6975 50  0000 L CNN
+F 2 "MyJacks:RCJ-2223" H 15100 6575 50  0001 C CNN
 F 3 " ~" H 15100 6575 50  0001 C CNN
 F 4 "HAND" H 15100 6675 50  0001 C CNN "JLPCB#"
-F 5 "Vertical Stereo RCA-pin Jack (Upper=Left, Lower=Right) RCJ-2232,RCJ-2233" H 15100 6675 50  0001 C CNN "Description"
+F 5 "Vertical Stereo RCA-pin Jack (Upper=Right, Lower=Left) RCJ-2223" H 15100 6675 50  0001 C CNN "Description"
 	1    15100 6675
 	1    0    0    -1
@@
 F 3 "~" H 14700 3600 50  0001 C CNN
 F 4 "NOP" H 14700 3600 50  0001 C CNN "JLPCB#"
+F 5 "Nount Zero-R when Non-Lifting GND RCA-pin Output" H 14700 3600 50  0001 C CNN "Description"
 	1    14700 3600
 	-1   0    0    1
@@
 F 3 "~" H 7525 7700 50  0001 C CNN
 F 4 "NOP" H 7525 7700 50  0001 C CNN "JLPCB#"
+F 5 "Nount Zero-R when Non-Lifting GND RCA-pin Output" H 7525 7700 50  0001 C CNN "Description"
 	1    7525 7700
 	1    0    0    -1
@@
 F 3 "~" H 6125 4375 50  0001 C CNN
 F 4 "C21189" H 6125 4375 50  0001 C CNN "JLPCB#"
+F 5 "Move to R171 when never use of XLR" H 6125 4375 50  0001 C CNN "Description"
 	1    6125 4375
 	0    -1   -1   0
@@
 F 3 "~" H 7075 3575 50  0001 C CNN
 F 4 "NOP" H 7075 3575 50  0001 C CNN "JLPCB#"
+F 5 "Nount Zero-R when Non-Lifting GND RCA-pin Output" H 7075 3575 50  0001 C CNN "Description"
 	1    7075 3575
 	1    0    0    -1
@@
 F 3 "~" H 10075 5800 50  0001 C CNN
 F 4 "C1017" H 10075 5800 50  0001 C CNN "JLPCB#"
+F 5 "Filter for DAC Power Rail" H 10075 5800 50  0001 C CNN "Description"
 	1    10075 5800
 	-1   0    0    1
@@
 F 3 "~" H 10275 5800 50  0001 C CNN
 F 4 "C1017" H 10275 5800 50  0001 C CNN "JLPCB#"
+F 5 "Filter for DAC Power Rail" H 10275 5800 50  0001 C CNN "Description"
 	1    10275 5800
 	1    0    0    -1
@@
 F 3 "~" H 2425 5900 50  0001 C CNN
 F 4 "C1017" H 2425 5900 50  0001 C CNN "JLPCB#"
+F 5 "Filter for DAC Power Rail" H 2425 5900 50  0001 C CNN "Description"
 	1    2425 5900
 	-1   0    0    1
@@
 F 3 "~" H 2625 5900 50  0001 C CNN
 F 4 "C1017" H 2625 5900 50  0001 C CNN "JLPCB#"
+F 5 "Filter for DAC Power Rail" H 2625 5900 50  0001 C CNN "Description"
 	1    2625 5900
 	1    0    0    -1
@@
 F 3 "~" H 9975 1875 50  0001 C CNN
 F 4 "C1017" H 9975 1875 50  0001 C CNN "JLPCB#"
+F 5 "Filter for DAC Power Rail" H 9975 1875 50  0001 C CNN "Description"
 	1    9975 1875
 	-1   0    0    1
@@
 F 3 "~" H 10175 1875 50  0001 C CNN
 F 4 "C1017" H 10175 1875 50  0001 C CNN "JLPCB#"
+F 5 "Filter for DAC Power Rail" H 10175 1875 50  0001 C CNN "Description"
 	1    10175 1875
 	1    0    0    -1
@@
 P 7375 2875
 F 0 "J17" H 7300 3125 50  0000 L CNN
-F 1 "MJ-519" H 7250 3275 50  0000 L CNN
-F 2 "MyJacks:MJ-519" H 7375 2775 50  0001 C CNN
+F 1 "RCJ-2223" H 7250 3275 50  0000 L CNN
+F 2 "MyJacks:RCJ-2223" H 7375 2775 50  0001 C CNN
 F 3 " ~" H 7375 2775 50  0001 C CNN
 F 4 "HAND" H 7375 2875 50  0001 C CNN "JLPCB#"
-F 5 "Vertical Stereo RCA-pin Jack (Upper=Left, Lower=Right) RCJ-2232,RCJ-2233" H 7375 2875 50  0001 C CNN "Description"
+F 5 "Vertical Stereo RCA-pin Jack (Upper=Right, Lower=Left) RCJ-2223" H 7375 2875 50  0001 C CNN "Description"
 	1    7375 2875
 	1    0    0    -1
@@
 F 3 "~" H 2200 1975 50  0001 C CNN
 F 4 "C1017" H 2200 1975 50  0001 C CNN "JLPCB#"
+F 5 "Filter for DAC Power Rail" H 2200 1975 50  0001 C CNN "Description"
 	1    2200 1975
 	-1   0    0    1
@@
 F 3 "~" H 2400 1975 50  0001 C CNN
 F 4 "C1017" H 2400 1975 50  0001 C CNN "JLPCB#"
+F 5 "Filter for DAC Power Rail" H 2400 1975 50  0001 C CNN "Description"
 	1    2400 1975
 	1    0    0    -1
@@
 F 3 "~" H 6550 8400 50  0001 C CNN
 F 4 "C21189" H 6550 8400 50  0001 C CNN "JLPCB#"
+F 5 "Move to R213 when never use of XLR" H 6550 8400 50  0001 C CNN "Description"
 	1    6550 8400
 	0    1    1    0
@@
 DAC3_R
 Text Notes 15000 2875 0    63   ~ 0
-OUT-32\n(RIGHT)\nOUT-33\n(LEFT)
+OUT-33\n(RIGHT)\nOUT-32\n(LEFT)\n
 Text Notes 15200 6900 0    63   ~ 0
-OUT-40\n(RIGHT)\nOUT-41\n(LEFT)
-Text Notes 7850 6900 0    63   ~ 0
-OUT-16\n(RIGHT)\nOUT-17\n(LEFT)
+OUT-41\n(RIGHT)\nOUT-40\n(LEFT)\n
+Text Notes 7850 7000 0    63   ~ 0
+OUT-17\n(RIGHT)\nOUT-16\n(LEFT)
 Wire Wire Line
 	7075 4075 7125 4075
@@
 F 3 "~" H 14175 8150 50  0001 C CNN
 F 4 "C21189" H 14175 8150 50  0001 C CNN "JLPCB#"
+F 5 "Move to R212 when never use of XLR" H 14175 8150 50  0001 C CNN "Description"
 	1    14175 8150
 	0    -1   -1   0
@@
 AR Path="/5D902CF8/6687663F" Ref="C?"  Part="1"
 AR Path="/5D902CF8/65D81CA2/6687663F" Ref="C147"  Part="1"
-F 0 "C147" V 12375 7275 50  0000 C CNN
+F 0 "C147" V 12250 7350 50  0000 C CNN
 F 1 "NOP" V 12325 7375 50  0000 C CNN
 F 2 "Capacitor_SMD:C_0805_2012Metric_Pad1.18x1.45mm_HandSolder" H 12425 7375 50  0001 C CNN
@@
 F 3 "~" H 14875 7425 50  0001 C CNN
 F 4 "NOP" H 14875 7425 50  0001 C CNN "JLPCB#"
+F 5 "Nount Zero-R when Non-Lifting GND RCA-pin Output" H 14875 7425 50  0001 C CNN "Description"
 	1    14875 7425
 	1    0    0    -1
@@
 F 3 "~" H 14025 4300 50  0001 C CNN
 F 4 "C21189" H 14025 4300 50  0001 C CNN "JLPCB#"
+F 5 "Move to R172 when never use of XLR" H 14025 4300 50  0001 C CNN "Description"
 	1    14025 4300
 	0    -1   -1   0
@@
 	11025 4300 11175 4300
 Connection ~ 14275 3225
-Text Notes 7475 3025 0    63   ~ 0
-OUT-0\n(RIGHT)\nOUT-1\n(LEFT)
+Text Notes 7475 3075 0    63   ~ 0
+OUT-1\n(RIGHT)\nOUT-0\n(LEFT)\n
 $Comp
 L Device:C_Small C?
@@
 Text Label 3725 6650 0    50   ~ 0
 DAC1_R
-Text Label 6850 2775 0    50   ~ 0
-OUT0_P
-Text Label 6850 2975 0    50   ~ 0
-OUT1_P
 Text Label 6900 3225 0    50   ~ 0
 DIFF_GND0
@@
 	6275 4375 6350 4375
 Wire Wire Line
-	6750 2175 6750 2975
-Connection ~ 6750 2975
-Wire Wire Line
-	6750 2975 6750 3875
-Wire Wire Line
-	6450 2775 6450 3325
-Wire Wire Line
-	6750 2975 7175 2975
-Wire Wire Line
-	6450 2775 7175 2775
-Wire Wire Line
 	3200 2725 3675 2725
 Connection ~ 3200 2725
@@
 	3700 6550 4200 6550
 Wire Wire Line
-	14575 2750 14700 2750
-Connection ~ 14575 2750
-Wire Wire Line
-	14575 2750 14575 3800
-Wire Wire Line
-	14575 1950 14575 2750
-Wire Wire Line
-	14700 2550 14650 2550
-Wire Wire Line
-	14650 2550 14650 3225
-Wire Wire Line
 	14650 3225 14275 3225
 Wire Wire Line
@@
 	6350 4375 7075 4375
 Wire Wire Line
-	6550 2650 6550 4075
-Wire Wire Line
 	6550 4075 7075 4075
 Wire Wire Line
@@
 fc=87kHz
 Text Notes 15050 6325 0    50   ~ 0
-CUI RCJ-2232(2233)
+CUI
 Text Notes 14850 2300 0    50   ~ 0
-CUI RCJ-2232(2233)
+CUI
 Text Notes 7250 2450 0    50   ~ 0
-CUI RCJ-2232(2233)
+CUI
 Text Notes 7525 6400 0    50   ~ 0
-CUI RCJ-2232(2233)
+CUI
+Wire Wire Line
+	6550 2650 6550 4075
+Wire Wire Line
+	6750 2975 7175 2975
+Text Label 6825 2975 0    50   ~ 0
+OUT0_P
+Text Label 6825 2775 0    50   ~ 0
+OUT1_P
+Connection ~ 6750 2975
+Wire Wire Line
+	6750 2975 6750 3875
+Wire Wire Line
+	6750 2175 6750 2975
+Wire Wire Line
+	7175 2775 6450 2775
+Wire Wire Line
+	6450 2775 6450 3325
+Wire Wire Line
+	14575 1950 14575 2750
+Wire Wire Line
+	14700 2750 14575 2750
+Connection ~ 14575 2750
+Wire Wire Line
+	14575 2750 14575 3800
+Wire Wire Line
+	14700 2550 14650 2550
+Wire Wire Line
+	14650 3225 14650 2550
 $EndSCHEMATC
