File: SOURCES/kiCAD/DAC.sch (KiCad schematic (older format))
At the start: 196 parts, among them J16 RCJ-2223, J17 RCJ-2223, J20 RCJ-2223, J21 RCJ-2223, J24 Conn_01x06, J25 Conn_01x06, J27 Conn_01x06, J28 Conn_01x06, Q10 2SC3326, Q11 2SC3326, Q15 2SC3326, Q16 2SC3326, Q17 2SC3326, Q18 2SC3326, Q19 2SC3326, Q20 2SC3326, Q21 2SC3326, Q22 2SC3326, Q23 2SC3326, Q24 2SC3326, Q25 2SC3326, Q26 2SC3326, Q27 2SC3326, Q28 2SC3326, U14 PCM5102A, U16 PCM5102A, U17 PCM5102A, U18 PCM5102A, U20 OPA1632DR, U21 OPA1632DR, U22 OPA1632DR, U23 OPA1632DR, U24 OPA1632DR, U25 OPA1632DR, U26 OPA1632DR, U27 OPA1632DR

Commit message: A method of board type convertion had changed.
Add an AGND fill on the bottom layer. The connection path for the Standard type board had changed. No features/functions changed.
Parts:
- R136: renamed from C163; footprint Capacitor_SMD:C_0805_2012Metric_Pad1.18x1.45mm_HandSolder -> Resistors_SMD:R_0603_HandSoldering; symbol Device:C_Small -> Device:R
- R143: renamed from C162; footprint Capacitor_SMD:C_0805_2012Metric_Pad1.18x1.45mm_HandSolder -> Resistors_SMD:R_0603_HandSoldering; symbol Device:C_Small -> Device:R
- R147: renamed from C153; footprint Capacitor_SMD:C_0805_2012Metric_Pad1.18x1.45mm_HandSolder -> Resistors_SMD:R_0603_HandSoldering; symbol Device:C_Small -> Device:R
- R149: renamed from C152; footprint Capacitor_SMD:C_0805_2012Metric_Pad1.18x1.45mm_HandSolder -> Resistors_SMD:R_0603_HandSoldering; symbol Device:C_Small -> Device:R
- R157: renamed from C148; footprint Capacitor_SMD:C_0805_2012Metric_Pad1.18x1.45mm_HandSolder -> Resistors_SMD:R_0603_HandSoldering; symbol Device:C_Small -> Device:R
- R158: renamed from C147; footprint Capacitor_SMD:C_0805_2012Metric_Pad1.18x1.45mm_HandSolder -> Resistors_SMD:R_0603_HandSoldering; symbol Device:C_Small -> Device:R
- R171, R172, R212, R213: footprint Resistor_SMD:R_0603_1608Metric -> Resistor_SMD:R_0603_1608Metric_Pad0.98x0.95mm_HandSolder
- R66: renamed from C155; footprint Capacitor_SMD:C_0805_2012Metric_Pad1.18x1.45mm_HandSolder -> Resistors_SMD:R_0603_HandSoldering; symbol Device:C_Small -> Device:R
- R70: renamed from C156; footprint Capacitor_SMD:C_0805_2012Metric_Pad1.18x1.45mm_HandSolder -> Resistors_SMD:R_0603_HandSoldering; symbol Device:C_Small -> Device:R
Connections:
- net DAC0_L: now also R66.1
- net DAC0_R: now also R70.1
- net DAC1_L: now also R136.1
- net DAC1_R: now also R143.1
- net DAC2_L: now also R147.1
- net DAC2_R: now also R149.1
- net DAC3_L: now also R157.1
- net DAC3_R: now also R158.1
- net OUT0_P: now also R66.2
- net OUT16_P: now also R136.2
- net OUT17_P: now also R143.2
- net OUT1_P: now also R70.2
- net OUT32_P: now also R147.2
- net OUT33_P: now also R149.2
- net OUT40_P: now also R157.2
- net OUT41_P: now also R158.2
- net at R132.1, U20.1 (IN-): no longer R66.1
- net at R155.1, U20.4 (OUT+): no longer R66.2
- net at R134.1, U21.1 (IN-): no longer R70.1
- net at R156.2, U21.4 (OUT+): no longer R70.2
- net at R140.1, U24.1 (IN-): no longer R147.1
- net at R161.1, U24.4 (OUT+): no longer R147.2
- net at R142.1, U25.1 (IN-): no longer R149.1
- net at R162.2, U25.4 (OUT+): no longer R149.2
- net at R173.1, U26.1 (IN-): no longer R157.1
- net at R192.1, U26.4 (OUT+): no longer R157.2
- net at R175.1, U27.1 (IN-): no longer R158.1
- net at R194.2, U27.4 (OUT+): no longer R158.2
- net at R181.1, U22.1 (IN-): no longer R136.1
- net at R203.1, U22.4 (OUT+): no longer R136.2
- net at R183.1, U23.1 (IN-): no longer R143.1
- net at R204.2, U23.4 (OUT+): no longer R143.2
Other:
- note added: "REMOVE;\n R133, R135,\n R141, R146,\n R182, R187,\n R174, R176\n\nMOVE:\n (220R) R155 -> R60, (220R) R156 -> R70\n (220R) R161 -> R147, (220R) R162-> R149\n (220R) R203 -> R136, (220R) R204-> R143\n (220R) R192 -> R157, (220R) R194-> R158\n\nPOPLULATE:\n (Zero R) R171, R172, R212, R213"
- note added: "REMOVE;\n U20, U21, U22, U23, U24, U25, U26, U27,\n Q16, Q18, Q27, Q28, Q19, Q20, Q23, Q24\n R132, R133, R134, R135, R137, R139, R151, R153, \n R140, R141, R142, R146, R148, R150, R144, R145, \n R181, R182, R183, R187, R184, R185, R189, R191,\n R173, R174, R175, R176, R177, R52, R178, R180,\n R152, R155, R154, R156, R166, R168,\n R161, R160, R162, R159, R169, R170,\n R203, R198, R204, R201, R210,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"
- note added: "To Convert FreeDSP OVTAVIA DIFF/BAL version to Basic version."
- note added: "To Order FreeDSP OVTAVIA Basic version Example"
- note removed: "AS WELL TO THE ANOTHER PART …"
- note removed: "REMOVE;\n U26, U27, Q21, Q22, R202, R205, R173, R175, R194, R192, C145\n\nCHANGE:\n (to 0R) R174, R178, R193, R176, R180, R195, R177, R52\n\nJUMPER:\n Between J27 pin6-pin5, Between J27 pin2-pin3"
- note removed: "To Create FreeDSP OVTAVIA Basic version Example"
- moved on the sheet: C127, C128, C129, C130, C135, C136, C137, C138, C157, J17, Q10, Q16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
